Commit message: Add S2 Integration and child_link update

File: urdf/spherical_pendulum.urdf.xacro (robot description, xacro)
@@ -67,8 +67,4 @@
         <parent link="fixed_base"/>
         <child link="cable"/>
-<!--        <calibration rising="0.0"/>-->
-<!--        <dynamics damping="0.0" friction="0.0"/>-->
-<!--        <limit effort="30" velocity="1.0" lower="-2.2" upper="0.7" />-->
-<!--        <safety_controller k_velocity="10"/>-->
     </joint>
     <!--    <gazebo>-->

Commit message: Create universal joint in plugin

File: urdf/spherical_pendulum.urdf.xacro (robot description, xacro)
@@ -50,10 +50,10 @@
             <origin xyz="0 0 ${cable_length/2}" rpy="0 0 0"/>
             <geometry>
-                <cylinder length="${cable_length}" radius="${2*cable_radius}"/>
+                <cylinder length="${cable_length}" radius="${cable_radius}"/>
             </geometry>
         </visual>
         <inertial>
             <origin xyz="0 0 ${cable_length/2}" rpy="0 0 0"/>
-            <mass value="0.5"/>
+            <mass value="50"/>
             <inertia ixx="0.0001" ixy="0.0" ixz="0.0" iyy="0.0001" iyz="0.0" izz="0.0004"/>
         </inertial>
@@ -68,12 +68,4 @@
         <child link="cable"/>
     </joint>
-    <!--    <gazebo>-->
-    <!--        <model name="universal_joint">-->
-    <!--            <joint name="joint" type="universal">-->
-    <!--                <parent>fixed_base</parent>-->
-    <!--                <child>cable</child>-->
-    <!--            </joint>-->
-    <!--        </model>-->
-    <!--    </gazebo>-->
     <!-- Macro to add a qrotor_sil plugin. -->
     <xacro:macro name="spherical_joint_plugin" params="namespace parent_link child_link">
@@ -87,64 +79,3 @@
     </xacro:macro>
     <xacro:spherical_joint_plugin namespace="spherical_pendulum" parent_link="fixed_base" child_link="cable"/>
-<!--    &lt;!&ndash; MACRO: dummy link to create 3D rotation (in Euler Angles) &ndash;&gt;-->
-<!--    <xacro:macro name="dummy_link" params="name">-->
-<!--        <link name="${name}">-->
-<!--            <gravity>0</gravity>-->
-<!--            <inertial>-->
-<!--                <origin rpy="0 0 0" xyz="0 0 0"/>-->
-<!--                <mass value="0.00001"/>-->
-<!--                <inertia ixx="0.000000001" ixy="0" ixz="0" iyy="0.000000001" iyz="0" izz="0.000000001"/>-->
-<!--            </inertial>-->
-<!--            <visual>-->
-<!--                <geometry>-->
-<!--                    <sphere radius="0.001"/>-->
-<!--                </geometry>-->
-<!--            </visual>-->
-<!--        </link>-->
-<!--        <gazebo reference="${name}">-->
-<!--            <material>Gazebo/Black</material>-->
-<!--        </gazebo>-->
-<!--    </xacro:macro>-->
-<!--    &lt;!&ndash; MACRO: create a rotational joint ( TODO: debug this joint) &ndash;&gt;-->
-<!--    <xacro:macro name="rotational_joint" params="parent child jx jy jz r p y">-->
-<!--        <xacro:dummy_link name="${parent}_${child}_dummylink1"/>-->
-<!--        <xacro:dummy_link name="${parent}_${child}_dummylink2"/>-->
-<!--        <joint name="${parent}_${child}_roll" type="continuous">-->
-<!--            <parent link="${parent}"/>-->
-<!--            <child link="${parent}_${child}_dummylink1"/>-->
-<!--            <axis xyz="1 0 0"/>-->
-<!--            &lt;!&ndash; <limit effort="1000.0" lower="0.0" upper="0.548" velocity="0.5"/> &ndash;&gt;-->
-<!--            <dynamics damping="0.0" friction="0.0"/>-->
-<!--            &lt;!&ndash; <limit effort="30" velocity="1.0" lower="-2.2" upper="0.7" />-->
-<!--            <safety_controller k_velocity="10" k_position="15" soft_lower_limit="-2.0" soft_upper_limit="0.5" /> &ndash;&gt;-->
-<!--            &lt;!&ndash; <joint_properties damping="0.0" friction="0.0" /> &ndash;&gt;-->
-<!--            <origin xyz="${jx} ${jy} ${jz}" rpy="${r} 0 0"/>-->
-<!--        </joint>-->
-<!--        <joint name="${parent}_${child}_pitch" type="continuous">-->
-<!--            <parent link="${parent}_${child}_dummylink1"/>-->
-<!--            <child link="${parent}_${child}_dummylink2"/>-->
-<!--            <axis xyz="0 1 0"/>-->
-<!--            &lt;!&ndash; <limit effort="1000.0" lower="0.0" upper="0.548" velocity="0.5"/> &ndash;&gt;-->
-<!--            <dynamics damping="0.0" friction="0.0"/>-->
-<!--            &lt;!&ndash; <dynamics damping="0.0" friction="0.0"/>-->
-<!--            <limit effort="30" velocity="1.0" lower="-2.2" upper="0.7" />-->
-<!--            <safety_controller k_velocity="10" k_position="15" soft_lower_limit="-2.0" soft_upper_limit="0.5" /> &ndash;&gt;-->
-<!--            &lt;!&ndash; <joint_properties damping="0.0" friction="0.0" /> &ndash;&gt;-->
-<!--            <origin xyz="0 0 0" rpy="0 ${p} 0"/>-->
-<!--        </joint>-->
-<!--        <joint name="${parent}_${child}_yaw" type="continuous">-->
-<!--            <parent link="${parent}_${child}_dummylink2"/>-->
-<!--            <child link="${child}"/>-->
-<!--            <axis xyz="0 0 1"/>-->
-<!--            &lt;!&ndash; <limit effort="1000.0" lower="0.0" upper="0.548" velocity="0.5"/> &ndash;&gt;-->
-<!--            <dynamics damping="0.0" friction="0.0"/>-->
-<!--            &lt;!&ndash; <dynamics damping="0.0" friction="0.0"/> &ndash;&gt;-->
-<!--            &lt;!&ndash; <limit effort="30" velocity="1.0" lower="-2.2" upper="0.7" /> &ndash;&gt;-->
-<!--            &lt;!&ndash; <safety_controller k_velocity="10" k_position="15" soft_lower_limit="-2.0" soft_upper_limit="0.5" /> &ndash;&gt;-->
-<!--            &lt;!&ndash; <joint_properties damping="0.0" friction="0.0" /> &ndash;&gt;-->
-<!--            <origin xyz="0 0 0" rpy="0 0 ${y}"/>-->
-<!--        </joint>-->
-<!--    </xacro:macro>-->
-<!--    <xacro:rotational_joint parent="fixed_base" child="cable" jx="0" jy="0" jz="${-base_height/2}" r="${PI/2}"-->
-<!--                            p="${PI/4}" y="${PI/4}"/>-->
 </robot>

Commit message: Fix joint name (no longer hardcoded) and test two spherical joints

File: urdf/spherical_pendulum.urdf.xacro (robot description, xacro)
@@ -4,5 +4,5 @@
     <!-- Constants for robot dimensions -->
     <xacro:property name="PI" value="3.1415926535897931"/>
-    <xacro:property name="mass" value="1"/>
+    <xacro:property name="mass" value="10"/>
     <xacro:property name="base_width" value="0.5"/>
     <xacro:property name="base_length" value="0.5"/>
@@ -10,4 +10,15 @@
     <xacro:property name="cable_length" value="1"/>
     <xacro:property name="cable_radius" value="0.002"/>
+    <xacro:property name="cable_mass" value="0.1"/>
+    <!-- Macro to add a spherical_joint_plugin. -->
+    <xacro:macro name="spherical_joint_plugin" params="namespace parent_link child_link">
+        <gazebo>
+            <plugin filename="libspherical_joint_plugin.so" name="spherical_joint_plugin">
+                <parent_link>${parent_link}</parent_link>
+                <child_link>${child_link}</child_link>
+                <namespace>${namespace}</namespace>
+            </plugin>
+        </gazebo>
+    </xacro:macro>
     <!-- Used for fixing robot to Gazebo 'base_link' -->
     <link name="world"/>
@@ -37,4 +48,5 @@
         </inertial>
     </link>
+    <!-- Cable Link -->
     <link name="cable">
         <collision>
@@ -55,5 +67,5 @@
         <inertial>
             <origin xyz="0 0 ${cable_length/2}" rpy="0 0 0"/>
-            <mass value="50"/>
+            <mass value="${cable_mass}"/>
             <inertia ixx="0.0001" ixy="0.0" ixz="0.0" iyy="0.0001" iyz="0.0" izz="0.0004"/>
         </inertial>
@@ -63,19 +75,36 @@
         <self_collide>0</self_collide>
     </gazebo>
-    <joint name="dummy_spherical_joint" type="floating">
+    <!-- Payload Link -->
+    <link name="payload">
+        <collision>
+            <origin xyz="0 0 0" rpy="0 0 0"/>
+            <geometry>
+                <box size="${base_length} ${base_width} ${base_height}"/>
+            </geometry>
+        </collision>
+        <visual>
+            <origin xyz="0 0 0" rpy="0 0 0"/>
+            <geometry>
+                <box size="${base_length} ${base_width} ${base_height}"/>
+            </geometry>
+            <material name="orange"/>
+        </visual>
+        <inertial>
+            <origin xyz="0 0 0" rpy="0 0 0"/>
+            <mass value="${mass}"/>
+            <inertia ixx="0.001" ixy="0.0" ixz="0.0" iyy="0.001" iyz="0.0" izz="0.001"/>
+        </inertial>
+    </link>
+    <joint name="dummy_fixed_base_cable_joint" type="floating">
         <origin xyz="0 0 ${-base_height/2}" rpy="${PI/2} ${PI/4} ${PI/4}"/>
         <parent link="fixed_base"/>
         <child link="cable"/>
     </joint>
-    <!-- Macro to add a qrotor_sil plugin. -->
-    <xacro:macro name="spherical_joint_plugin" params="namespace parent_link child_link">
-        <gazebo>
-            <plugin filename="libspherical_joint_plugin.so" name="spherical_joint_plugin">
-                <parent_link>${parent_link}</parent_link>
-                <child_link>${child_link}</child_link>
-                <namespace>${namespace}</namespace>
-            </plugin>
-        </gazebo>
-    </xacro:macro>
-    <xacro:spherical_joint_plugin namespace="spherical_pendulum" parent_link="fixed_base" child_link="cable"/>
+    <joint name="dummy_cable_payload_joint" type="floating">
+        <origin xyz="0 0 ${cable_length}" rpy="0 0 0"/>
+        <parent link="cable"/>
+        <child link="payload"/>
+    </joint>
+    <xacro:spherical_joint_plugin namespace="joint1" parent_link="fixed_base" child_link="cable"/>
+    <xacro:spherical_joint_plugin namespace="joint2" parent_link="cable" child_link="payload"/>
 </robot>
